Commit message: Corrected model with quadrotor as root
Previous commit was based off of an incorrect urdf file for the 2DOF aerial manipulator, so this commit makes modifications to the correct file (uam_2dof.urdf) that have the vehicle base as the root joint

File: models/uam_2dof_pin.urdf (robot description, URDF)
Before this commit: robot AerialManipulator, 14 links, 13 joints
Links:
- link COM: mass None -> 1e-10
- link arm: mass None -> 1e-10
- link gripper: mass None -> 1e-10
- link motor1: mass None -> 1e-10
- link motor2: mass None -> 1e-10
- link motor3: mass None -> 1e-10
- link motor4: mass None -> 1e-10
- link prop1: mass None -> 1e-10
- link prop2: mass None -> 1e-10
- link prop3: mass None -> 1e-10
- link prop4: mass None -> 1e-10
- link virtualvehicle: mass None -> 1e-10
Joints:
- joint com_placement: origin xyz=0 0 -0.05 rpy=0 0 0 -> xyz=0 0 -0.041 rpy=0 0 0

File: models/uam_2dof_pin_continuous.urdf (robot description, URDF)
Before this commit: robot AerialManipulator, 14 links, 13 joints
Links:
- link COM: mass None -> 1e-10
- link arm: mass None -> 1e-10
- link gripper: mass None -> 1e-10
- link motor1: mass None -> 1e-10
- link motor2: mass None -> 1e-10
- link motor3: mass None -> 1e-10
- link motor4: mass None -> 1e-10
- link prop1: mass None -> 1e-10
- link prop2: mass None -> 1e-10
- link prop3: mass None -> 1e-10
- link prop4: mass None -> 1e-10
- link virtualvehicle: mass None -> 1e-10
Joints:
- joint com_placement: origin xyz=0 0 -0.05 rpy=0 0 0 -> xyz=0 0 -0.041 rpy=0 0 0
