Commit message: writing now

File: models/uam_2dof_ee_mass.urdf (robot description, URDF)
Before this commit: robot AerialManipulator, 14 links, 13 joints
Links:
- added link endeffector_com, mass 0.2; visual sphere radius=0.01
- link endeffector: geometry visual sphere radius=0.01
Joints:
- added joint endeffector_com_placement: type fixed, parent endeffector, child endeffector_com, origin xyz=0 -0.1 0 rpy=-1.57079632679 0 0
- joint joint_shoulder: limit lower=-3.14159265359 upper=3.14159265359 effort=2.0 velocity=1e9 -> lower=-31.4159265359 upper=31.4159265359 effort=2.0 velocity=1e9
- joint joint_wrist: limit lower=-3.14159265359 upper=3.14159265359 effort=1.0 velocity=1e9 -> lower=-31.4159265359 upper=31.4159265359 effort=1.0 velocity=1e9; origin xyz=0 0 -0.205 rpy=1.57079632679 3.14159265359 0 -> xyz=0 0 -0.205 rpy=1.57079632679 3.14159265359 1.57079632679

File: models/uam_2dof_ee_mass_pin.urdf (robot description, URDF)
Before this commit: robot AerialManipulator, 14 links, 13 joints
Links:
- added link endeffector_com, mass 0.2; visual sphere radius=0.01
- link COM: mass 1e-10 -> 1e-6
- link arm: mass 1e-10 -> 1e-6
- link endeffector: mass 0.2 -> 1e-6; geometry visual sphere radius=0.01
- link gripper: mass 1e-10 -> 1e-6
- link motor1: mass 1e-10 -> 1e-6
- link motor2: mass 1e-10 -> 1e-6
- link motor3: mass 1e-10 -> 1e-6
- link motor4: mass 1e-10 -> 1e-6
- link prop1: mass 1e-10 -> 1e-6
- link prop2: mass 1e-10 -> 1e-6
- link prop3: mass 1e-10 -> 1e-6
- link prop4: mass 1e-10 -> 1e-6
- link virtualvehicle: mass 1e-10 -> 1e-6
Joints:
- added joint endeffector_com_placement: type fixed, parent endeffector, child endeffector_com, origin xyz=0 -0.1 0 rpy=-1.57079632679 0 0
- joint joint_shoulder: limit lower=-3.14159265359 upper=3.14159265359 effort=2.0 velocity=1e9 -> lower=-31.4159265359 upper=31.4159265359 effort=2.0 velocity=1e9; type continuous -> revolute
- joint joint_wrist: limit lower=-3.14159265359 upper=3.14159265359 effort=1.0 velocity=1e9 -> lower=-31.4159265359 upper=31.4159265359 effort=1.0 velocity=1e9; origin xyz=0 0 -0.205 rpy=1.57079632679 3.14159265359 0 -> xyz=0 0 -0.205 rpy=1.57079632679 3.14159265359 1.57079632679; type continuous -> revolute
